File: electronics/remotetool/remotetool.sch (EAGLE design)
At the start: 48 parts

Commit message: remotetool: rename second half as it should be
The second half of connectors is kind of mirrored from the optocoupler
point of view; rename signals so that all connectors are facing the same
way when installing. Also make the borrom row labels readable.
Connections:
- net FOCUS10: now also NUCLEO2.28, R20.1; no longer NUCLEO2.26, R19.1
- net FOCUS6: now also NUCLEO2.4, R12.1; no longer NUCLEO2.2, R11.1
- net FOCUS7: now also NUCLEO2.12, R14.1; no longer NUCLEO2.6, R13.1
- net FOCUS8: now also NUCLEO2.16, R16.1; no longer NUCLEO2.14, R15.1
- net FOCUS9: now also NUCLEO2.24, R18.1; no longer NUCLEO2.22, R17.1
- net SHUTTER10: now also NUCLEO2.26, R19.1; no longer NUCLEO2.28, R20.1
- net SHUTTER6: now also NUCLEO2.2, R11.1; no longer NUCLEO2.4, R12.1
- net SHUTTER7: now also NUCLEO2.6, R13.1; no longer NUCLEO2.12, R14.1
- net SHUTTER8: now also NUCLEO2.14, R15.1; no longer NUCLEO2.16, R16.1
- net SHUTTER9: now also NUCLEO2.22, R17.1; no longer NUCLEO2.24, R18.1
